File: hardware/cryosentinel.kicad_pcb (KiCad board)
At the start: 2 copper layers, 0 parts

Commit message: chore: replace placeholder schematic/PCB with authentic base layout and regenerate KiCad exports
Parts:
- added AE1: Antenna_Loop, footprints:ANT_NFC_30x40, F.Cu at (94.5, 49.0)
- added BT1: 2xAAA, Battery:BatteryHolder_Keystone_2468_2xAAA, B.Cu at (86.0, 93.0)
- added C1: 12p, Capacitor_SMD:C_0805_2012Metric_Pad1.18x1.45mm_HandSolder, F.Cu at (84.1, 79.8)
- added C10: 100n, Capacitor_SMD:C_0805_2012Metric_Pad1.18x1.45mm_HandSolder, F.Cu at (86.1, 52.3)
- added C11: 1u, Capacitor_SMD:C_0805_2012Metric_Pad1.18x1.45mm_HandSolder, F.Cu at (74.5, 85.3)
- added C12: 4n7, Capacitor_SMD:C_0805_2012Metric_Pad1.18x1.45mm_HandSolder, F.Cu at (68.6, 94.5)
- added C13: 100n, Capacitor_SMD:C_0805_2012Metric_Pad1.18x1.45mm_HandSolder, F.Cu at (81.2, 67.3)
- added C14: 10u, Capacitor_SMD:C_0805_2012Metric_Pad1.18x1.45mm_HandSolder, F.Cu at (81.2, 65.3)
- added C15: 100n, Capacitor_SMD:C_0805_2012Metric_Pad1.18x1.45mm_HandSolder, F.Cu at (70.6, 51.3)
- added C16: 100n, Capacitor_SMD:C_0805_2012Metric_Pad1.18x1.45mm_HandSolder, F.Cu at (68.3, 55.4)
- added C18: 10u, Capacitor_SMD:C_0805_2012Metric_Pad1.18x1.45mm_HandSolder, F.Cu at (90.1, 74.2)
- added C19: 100n, Capacitor_SMD:C_0805_2012Metric_Pad1.18x1.45mm_HandSolder, F.Cu at (90.2, 76.2)
- added C2: 12p, Capacitor_SMD:C_0805_2012Metric_Pad1.18x1.45mm_HandSolder, F.Cu at (84.1, 75.9)
- added C20: 100n, Capacitor_SMD:C_0805_2012Metric_Pad1.18x1.45mm_HandSolder, F.Cu at (90.2, 71.1)
- added C21: 100n, Capacitor_SMD:C_0805_2012Metric_Pad1.18x1.45mm_HandSolder, F.Cu at (68.3, 51.3)
- added C3: 22u, Capacitor_SMD:C_1206_3216Metric_Pad1.33x1.80mm_HandSolder, F.Cu at (86.9, 64.7)
- added C4: 100n, Capacitor_SMD:C_0805_2012Metric_Pad1.18x1.45mm_HandSolder, F.Cu at (84.4, 64.2)
- added C5: 10u, Capacitor_SMD:C_0805_2012Metric_Pad1.18x1.45mm_HandSolder, F.Cu at (68.6, 90.4)
- added C6: 100n, Capacitor_SMD:C_0805_2012Metric_Pad1.18x1.45mm_HandSolder, F.Cu at (90.8, 85.3)
- added C8: 100n, Capacitor_SMD:C_0805_2012Metric_Pad1.18x1.45mm_HandSolder, F.Cu at (70.4, 55.4)
- added C9: 100n, Capacitor_SMD:C_0805_2012Metric_Pad1.18x1.45mm_HandSolder, F.Cu at (76.7, 85.3)
- added D1: BAT60A, Diode_SMD:D_SOD-323_HandSoldering, F.Cu at (62.0, 86.4)
- added D2: LED, LED_SMD:LED_0805_2012Metric_Pad1.15x1.40mm_HandSolder, F.Cu at (63.0, 69.0)
- added D3: PRTR5V0U2X, Package_TO_SOT_SMD:SOT-143, F.Cu at (62.7, 83.6)
- added F1: MSMF010 0.01A, Fuse:Fuse_1812_4532Metric_Pad1.30x3.40mm_HandSolder, F.Cu at (90.7, 93.2)
- added FB1: 330, Resistor_SMD:R_0805_2012Metric_Pad1.20x1.40mm_HandSolder, F.Cu at (81.2, 63.2)
- added G***: LOGO, LOGO, F.Cu at (92.6, 64.1)
- added G04: LOGO, LOGO, F.Cu at (109.5, 64.0)
- added H1: MountingHole_Pad, MountingHole:MountingHole_3.2mm_M3_Pad_Via, F.Cu at (62.5, 44.5)
- added H2: MountingHole_Pad, MountingHole:MountingHole_3.2mm_M3_Pad_Via, F.Cu at (121.5, 44.5)
- added H3: MountingHole_Pad, MountingHole:MountingHole_3.2mm_M3_Pad_Via, F.Cu at (121.5, 93.5)
- added H4: MountingHole_Pad, MountingHole:MountingHole_3.2mm_M3_Pad_Via, F.Cu at (62.5, 93.5)
- added J1: Pickit 5 Conn, Connector_PinSocket_2.54mm:PinSocket_1x08_P2.54mm_Vertical, F.Cu at (114.8, 93.5)
- added J2: USB Type-C, Connector_USB:USB_C_Receptacle_XKB_U262-16XN-4BVC11, B.Cu at (61.0, 84.0)
- added NT1: NetTie_2, NetTie:NetTie-2_SMD_Pad0.5mm, F.Cu at (72.4, 48.5)
- added NT2: NetTie_2, NetTie:NetTie-2_SMD_Pad0.5mm, F.Cu at (88.6, 72.6)
- added NT3: NetTie_2, NetTie:NetTie-2_SMD_Pad0.5mm, F.Cu at (83.8, 51.3)
- added NT4: NetTie_2, NetTie:NetTie-2_SMD_Pad0.5mm, F.Cu at (62.5, 55.4)
- added NT5: NetTie_2, NetTie:NetTie-2_SMD_Pad0.5mm, F.Cu at (63.8, 57.9)
- added Q1: IRLML6401, Package_TO_SOT_SMD:SOT-23, F.Cu at (82.3, 91.4)
- added R1: 10k, Resistor_SMD:R_0805_2012Metric_Pad1.20x1.40mm_HandSolder, F.Cu at (70.5, 85.3)
- added R10: 4k7, Resistor_SMD:R_0805_2012Metric_Pad1.20x1.40mm_HandSolder, F.Cu at (75.3, 62.1)
- added R2: 10k, Resistor_SMD:R_0805_2012Metric_Pad1.20x1.40mm_HandSolder, F.Cu at (72.5, 85.3)
- added R3: 1k, Resistor_SMD:R_0805_2012Metric_Pad1.20x1.40mm_HandSolder, F.Cu at (86.5, 85.3)
- added R4: 10k, Resistor_SMD:R_0805_2012Metric_Pad1.20x1.40mm_HandSolder, F.Cu at (88.6, 85.3)
- added R5: 1M, Resistor_SMD:R_0805_2012Metric_Pad1.20x1.40mm_HandSolder, F.Cu at (68.6, 92.5)
- added R6: 5k1, Resistor_SMD:R_0805_2012Metric_Pad1.20x1.40mm_HandSolder, F.Cu at (67.7, 87.5)
- added R7: 5k1, Resistor_SMD:R_0805_2012Metric_Pad1.20x1.40mm_HandSolder, F.Cu at (63.2, 76.5)
- added R8: 1k, Resistor_SMD:R_0805_2012Metric_Pad1.20x1.40mm_HandSolder, F.Cu at (63.2, 74.3)
- added R9: 4k7, Resistor_SMD:R_0805_2012Metric_Pad1.20x1.40mm_HandSolder, F.Cu at (77.3, 62.1)
- added REF**: KiCad-Logo2_5mm_SilkScreen, Symbol:KiCad-Logo2_5mm_SilkScreen, F.Cu at (109.6, 78.4)
- added TP1: TestPoint_Probe, TestPoint:TestPoint_THTPad_D1.5mm_Drill0.7mm, F.Cu at (83.6, 46.2)
- added TP11: TestPoint_Probe, TestPoint:TestPoint_THTPad_D1.5mm_Drill0.7mm, F.Cu at (68.3, 46.2)
- added TP2: TestPoint_Probe, TestPoint:TestPoint_THTPad_D1.5mm_Drill0.7mm, F.Cu at (86.4, 46.2)
- added TP6: TestPoint_Probe, TestPoint:TestPoint_THTPad_D1.5mm_Drill0.7mm, F.Cu at (89.2, 46.2)
- added TP8: TestPoint_Probe, TestPoint:TestPoint_THTPad_D1.5mm_Drill0.7mm, F.Cu at (81.8, 70.9)
- added TP9: TestPoint_Probe, TestPoint:TestPoint_THTPad_D1.5mm_Drill0.7mm, F.Cu at (81.8, 73.4)
- added U1: L78L33ABUTR, Package_TO_SOT_SMD:SOT-89-3_Handsoldering, F.Cu at (77.5, 93.2)
- added U2: ATSAMD21E18A-AU, Package_QFP:TQFP-32_7x7mm_P0.8mm, F.Cu at (74.7, 75.2)
- added U3: AT25DF321, Package_SO:SOP-8_5.28x5.23mm_P1.27mm, F.Cu at (71.1, 63.5)
- added U4: ATECC608A-MAHDA-S, Package_DFN_QFN:DFN-8-1EP_3x2mm_P0.5mm_EP1.3x1.5mm, F.Cu at (73.1, 51.4)
- added U6: SHT30-DIS, Sensor_Humidity:Sensirion_DFN-8-1EP_2.5x2.5mm_P0.5mm_EP1.1x1.7mm, F.Cu at (63.0, 61.0)
- added U7: MMA8452QR1, Personal:XDCR_MMA8452QR1, F.Cu at (85.9, 71.6)
- added U8: OPT3001DNPR, Personal:SON65P200X200X65-7N, F.Cu at (63.0, 53.0)
- added U9: ST25DV04K, Package_SO:TSSOP-8_4.4x3mm_P0.65mm, F.Cu at (88.1, 49.2)
- added Y1: SC-32S32.768, Crystal:Crystal_SMD_EuroQuartz_EQ161-2Pin_3.2x1.5mm_HandSoldering, F.Cu at (81.8, 77.7)
Routing:
- net +3V0: track 0.00 -> 206.7 mm
- net SCL: track 0.00 -> 106.4 mm, vias 0 -> 2
- net SDA: track 0.00 -> 102.8 mm, vias 0 -> 2
- net ~RESET: track 0.00 -> 97.0 mm, vias 0 -> 1
- net NFC_INT: track 0.00 -> 40.1 mm, vias 0 -> 1
- net +5V: track 0.00 -> 39.8 mm, vias 0 -> 3
- net SWDCLK: track 0.00 -> 35.6 mm, vias 0 -> 2
- net LIGHT_INT: track 0.00 -> 35.0 mm
- net SWDIO: track 0.00 -> 26.0 mm, vias 0 -> 1
- net ~TEMP_RESET: track 0.00 -> 23.3 mm
- net TEMP_INT: track 0.00 -> 22.1 mm, vias 0 -> 2
- net USB_D+: track 0.00 -> 16.0 mm, vias 0 -> 1
- net USB_D-: track 0.00 -> 15.3 mm, vias 0 -> 1
- net SCK: track 0.00 -> 14.9 mm, vias 0 -> 2
- net Net-(D3-GND): track 0.00 -> 13.8 mm
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- added copper zone on B.Cu, net GND
- added copper zone on F.Cu, net GND
Other:
- board outline added: 68 x 58 mm
- board text added: "2xAAA 2.4-3.0V"
- board text added: "3V"
- board text added: "CORTEX M0+"
- board text added: "CRYPTO"
- board text added: "FLASH"
- board text added: "GND"
- board text added: "IMU"
- board text added: "IMU_INT1"
- board text added: "IMU_INT2"
- board text added: "LIGHT"
- board text added: "LIGHT_INT"
- board text added: "MISO"
- board text added: "MOSI"
- board text added: "NFC"
- board text added: "NFC_INT"
- board text added: "PICKIT 5"
- board text added: "RISK DATA LOGGER"
- board text added: "SCK"
- board text added: "SCL"
- board text added: "SDA"
- board text added: "SN| |"
- board text added: "SWDCLK"
- board text added: "SWDIO"
- board text added: "TEMP"
- board text added: "USB-C"
- board text added: "by apolisskyi"
- board text added: "~CS"
- board text added: "~RESET"
