File: hardware/cryosentinel.kicad_pcb (KiCad board)
At the start: 2 copper layers, 68 x 58 mm, 66 parts, among them J1 Pickit 5 Conn, J2 USB Type-C, Q1 IRLML6401, U1 L78L33ABUTR, U2 ATSAMD21E18A-AU, U3 AT25DF321, U4 ATECC608A-MAHDA-S, U6 SHT30-DIS, U7 MMA8452QR1, U8 OPT3001DNPR, U9 ST25DV04K, Y1 SC-32S32.768

Commit message: hardware: complete CryoSentinel v2.0 schematic layout and 3D visualization
Parts:
- removed AE1: Antenna_Loop, footprints:ANT_NFC_30x40
- removed BT1: 2xAAA, Battery:BatteryHolder_Keystone_2468_2xAAA
- removed C1, C2: 12p, Capacitor_SMD:C_0805_2012Metric_Pad1.18x1.45mm_HandSolder
- removed C10, C13, C15, C16, C19, C20, C21, C4, C6, C8, C9: 100n, Capacitor_SMD:C_0805_2012Metric_Pad1.18x1.45mm_HandSolder
- removed C11: 1u, Capacitor_SMD:C_0805_2012Metric_Pad1.18x1.45mm_HandSolder
- removed C12: 4n7, Capacitor_SMD:C_0805_2012Metric_Pad1.18x1.45mm_HandSolder
- removed C14, C18, C5: 10u, Capacitor_SMD:C_0805_2012Metric_Pad1.18x1.45mm_HandSolder
- removed C3: 22u, Capacitor_SMD:C_1206_3216Metric_Pad1.33x1.80mm_HandSolder
- removed D1: BAT60A, Diode_SMD:D_SOD-323_HandSoldering
- removed D2: LED, LED_SMD:LED_0805_2012Metric_Pad1.15x1.40mm_HandSolder
- removed D3: PRTR5V0U2X, Package_TO_SOT_SMD:SOT-143
- removed F1: MSMF010 0.01A, Fuse:Fuse_1812_4532Metric_Pad1.30x3.40mm_HandSolder
- removed FB1: 330, Resistor_SMD:R_0805_2012Metric_Pad1.20x1.40mm_HandSolder
- removed G***, G04: LOGO, LOGO
- removed H1, H2, H3, H4: MountingHole_Pad, MountingHole:MountingHole_3.2mm_M3_Pad_Via
- removed J1: Pickit 5 Conn, Connector_PinSocket_2.54mm:PinSocket_1x08_P2.54mm_Vertical
- removed J2: USB Type-C, Connector_USB:USB_C_Receptacle_XKB_U262-16XN-4BVC11
- removed NT1, NT2, NT3, NT4, NT5: NetTie_2, NetTie:NetTie-2_SMD_Pad0.5mm
- removed Q1: IRLML6401, Package_TO_SOT_SMD:SOT-23
- removed R1, R2, R4: 10k, Resistor_SMD:R_0805_2012Metric_Pad1.20x1.40mm_HandSolder
- removed R10, R9: 4k7, Resistor_SMD:R_0805_2012Metric_Pad1.20x1.40mm_HandSolder
- removed R3, R8: 1k, Resistor_SMD:R_0805_2012Metric_Pad1.20x1.40mm_HandSolder
- removed R5: 1M, Resistor_SMD:R_0805_2012Metric_Pad1.20x1.40mm_HandSolder
- removed R6, R7: 5k1, Resistor_SMD:R_0805_2012Metric_Pad1.20x1.40mm_HandSolder
- removed REF**: KiCad-Logo2_5mm_SilkScreen, Symbol:KiCad-Logo2_5mm_SilkScreen
- removed TP1, TP11, TP2, TP6, TP8, TP9: TestPoint_Probe, TestPoint:TestPoint_THTPad_D1.5mm_Drill0.7mm
- removed U1: L78L33ABUTR, Package_TO_SOT_SMD:SOT-89-3_Handsoldering
- removed U2: ATSAMD21E18A-AU, Package_QFP:TQFP-32_7x7mm_P0.8mm
- removed U3: AT25DF321, Package_SO:SOP-8_5.28x5.23mm_P1.27mm
- removed U4: ATECC608A-MAHDA-S, Package_DFN_QFN:DFN-8-1EP_3x2mm_P0.5mm_EP1.3x1.5mm
- removed U6: SHT30-DIS, Sensor_Humidity:Sensirion_DFN-8-1EP_2.5x2.5mm_P0.5mm_EP1.1x1.7mm
- removed U7: MMA8452QR1, Personal:XDCR_MMA8452QR1
- removed U8: OPT3001DNPR, Personal:SON65P200X200X65-7N
- removed U9: ST25DV04K, Package_SO:TSSOP-8_4.4x3mm_P0.65mm
- removed Y1: SC-32S32.768, Crystal:Crystal_SMD_EuroQuartz_EQ161-2Pin_3.2x1.5mm_HandSoldering
Routing:
- net +3V0: track 206.7 -> 0.00 mm
- net SCL: track 106.4 -> 0.00 mm, vias 2 -> 0
- net SDA: track 102.8 -> 0.00 mm, vias 2 -> 0
- net ~RESET: track 97.0 -> 0.00 mm, vias 1 -> 0
- net NFC_INT: track 40.1 -> 0.00 mm, vias 1 -> 0
- net +5V: track 39.8 -> 0.00 mm, vias 3 -> 0
- net SWDCLK: track 35.6 -> 0.00 mm, vias 2 -> 0
- net LIGHT_INT: track 35.0 -> 0.00 mm
- net SWDIO: track 26.0 -> 0.00 mm, vias 1 -> 0
- net ~TEMP_RESET: track 23.3 -> 0.00 mm
- net TEMP_INT: track 22.1 -> 0.00 mm, vias 2 -> 0
- net USB_D+: track 16.0 -> 0.00 mm, vias 1 -> 0
- net USB_D-: track 15.3 -> 0.00 mm, vias 1 -> 0
- net SCK: track 14.9 -> 0.00 mm, vias 2 -> 0
- net Net-(D3-GND): track 13.8 -> 0.00 mm
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- removed copper zone on B.Cu, net GND
- removed copper zone on F.Cu, net GND
Other:
- board outline removed
- board text removed: "2xAAA 2.4-3.0V"
- board text removed: "3V"
- board text removed: "CORTEX M0+"
- board text removed: "CRYPTO"
- board text removed: "FLASH"
- board text removed: "GND"
- board text removed: "IMU"
- board text removed: "IMU_INT1"
- board text removed: "IMU_INT2"
- board text removed: "LIGHT"
- board text removed: "LIGHT_INT"
- board text removed: "MISO"
- board text removed: "MOSI"
- board text removed: "NFC"
- board text removed: "NFC_INT"
- board text removed: "PICKIT 5"
- board text removed: "RISK DATA LOGGER"
- board text removed: "SCK"
- board text removed: "SCL"
- board text removed: "SDA"
- board text removed: "SN| |"
- board text removed: "SWDCLK"
- board text removed: "SWDIO"
- board text removed: "TEMP"
- board text removed: "USB-C"
- board text removed: "by apolisskyi"
- board text removed: "~CS"
- board text removed: "~RESET"
