File: hardware/cryosentinel.kicad_sch (KiCad schematic)
At the start: 13 parts

Commit message: chore: replace placeholder schematic/PCB with authentic base layout and regenerate KiCad exports
Parts:
- removed D1: LED_RED_GPIO12, LED_SMD:LED_0603_1608Metric, symbol Device:LED
- removed D3: LED_BLUE_GPIO14, LED_SMD:LED_0603_1608Metric, symbol Device:LED
- removed D4: LED_BAT_GPIO15, LED_SMD:LED_0603_1608Metric, symbol Device:LED
- removed _TEMPLATE_C: C_TEMPLATE, symbol Device:C
- removed _TEMPLATE_D: LED_TEMPLATE, symbol Device:LED
- removed _TEMPLATE_R: R_TEMPLATE, symbol Device:R
- added AE1: Antenna_Loop, footprints:ANT_NFC_30x40, symbol Device:Antenna_Loop
- added BT1: 2xAAA, Battery:BatteryHolder_Keystone_2468_2xAAA, symbol Device:Battery
- added C1, C2: 22p, Capacitor_SMD:C_0805_2012Metric_Pad1.18x1.45mm_HandSolder, symbol Device:C
- added C10, C13, C15, C16, C18, C19, C20, C21, C4, C6, C8, C9: 100n, Capacitor_SMD:C_0805_2012Metric_Pad1.18x1.45mm_HandSolder, symbol Device:C
- added C11, C14, C5: 10u, Capacitor_SMD:C_0805_2012Metric_Pad1.18x1.45mm_HandSolder, symbol Device:C
- added C12: 4n7, Capacitor_SMD:C_0805_2012Metric_Pad1.18x1.45mm_HandSolder, symbol Device:C
- added C3: 22u, Capacitor_SMD:C_1206_3216Metric_Pad1.33x1.80mm_HandSolder, symbol Device:C
- added D1: BAT60A, Diode_SMD:D_SOD-323_HandSoldering, symbol Diode:BAT60A
- added D3: PRTR5V0U2X, Package_TO_SOT_SMD:SOT-143, symbol Power_Protection:PRTR5V0U2X
- added F1: MSMF010 0.01A, Fuse:Fuse_1812_4532Metric_Pad1.30x3.40mm_HandSolder, symbol Device:Polyfuse
- added FB1: 330, Resistor_SMD:R_0805_2012Metric_Pad1.20x1.40mm_HandSolder, symbol Device:FerriteBead_Small
- added H1, H2, H3, H4: MountingHole_Pad, MountingHole:MountingHole_3.2mm_M3_Pad_Via, symbol Mechanical:MountingHole_Pad
- added J1: Pickit 5 Conn, Connector_PinSocket_2.54mm:PinSocket_1x08_P2.54mm_Vertical, symbol Connector:Conn_01x08_Socket
- added J2: USB Type-C, Connector_USB:USB_C_Receptacle_XKB_U262-16XN-4BVC11, symbol Connector:USB_C_Receptacle_USB2.0
- added NT1, NT2, NT3, NT4, NT5: NetTie_2, NetTie:NetTie-2_SMD_Pad0.5mm, symbol Device:NetTie_2
- added Q1: IRLML6401, Package_TO_SOT_SMD:SOT-23, symbol Device:Q_PMOS_GSD
- added R10, R9: 4k7, Resistor_SMD:R_0805_2012Metric_Pad1.20x1.40mm_HandSolder, symbol Device:R
- added R7: 5k1, Resistor_SMD:R_0805_2012Metric_Pad1.20x1.40mm_HandSolder, symbol Device:R
- added R8: 1k, Resistor_SMD:R_0805_2012Metric_Pad1.20x1.40mm_HandSolder, symbol Device:R
- added TP1, TP11, TP2, TP6, TP8, TP9: TestPoint_Probe, TestPoint:TestPoint_THTPad_D1.5mm_Drill0.7mm, symbol Connector:TestPoint_Probe
- added U1: L78L33ABUTR, Package_TO_SOT_SMD:SOT-89-3_Handsoldering, symbol Regulator_Linear:L78L33_SOT89
- added U2: ATSAMD21E18A-AU, Package_QFP:TQFP-32_7x7mm_P0.8mm, symbol ATSAMD21E17A-AUT:ATSAMD21E17A-AUT
- added U3: AT25DF321, Package_SO:SOP-8_5.28x5.23mm_P1.27mm, symbol AT25DF041B-XMHN-B:AT25DF041B-XMHN-B
- added U4: ATECC608A-MAHDA-S, Package_DFN_QFN:DFN-8-1EP_3x2mm_P0.5mm_EP1.3x1.5mm, symbol Security:ATECC608A-SSHDA
- added U6: SHT30-DIS, Sensor_Humidity:Sensirion_DFN-8-1EP_2.5x2.5mm_P0.5mm_EP1.1x1.7mm, symbol Sensor_Humidity:SHT30-DIS
- added U7: MMA8452QR1, Personal:XDCR_MMA8452QR1, symbol MMA8452Q:MMA8452Q
- added U8: OPT3001DNPR, Personal:SON65P200X200X65-7N, symbol OPT3001DNPR:OPT3001DNPR
- added U9: ST25DV04K, Package_SO:TSSOP-8_4.4x3mm_P0.65mm, symbol ST25DV64K-IER8T3:ST25DV64K-IER8T3
- added Y1: SC-32S32.768, Crystal:Crystal_SMD_EuroQuartz_EQ161-2Pin_3.2x1.5mm_HandSoldering, symbol Device:Crystal
- D2: value LED_GREEN_GPIO13 -> LED; footprint LED_SMD:LED_0603_1608Metric -> LED_SMD:LED_0805_2012Metric_Pad1.15x1.40mm_HandSolder; LCSC Part (none) -> C84260; Part (none) -> NCD0805G1; URL (none) -> https://www.lcsc.com/product-detail/Light-Emitting-Diodes-L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
- R1, R2, R4: value 330 -> 10k; footprint Resistor_SMD:R_0603_1608Metric -> Resistor_SMD:R_0805_2012Metric_Pad1.20x1.40mm_HandSolder; LCSC Part (none) -> C84376; Part (none) -> RC0805FR-0710KL; URL (none) -> https://www.lcsc.com/product-detail/Chip-Resistor-Surface-M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
- R3: value 330 -> 1k; footprint Resistor_SMD:R_0603_1608Metric -> Resistor_SMD:R_0805_2012Metric_Pad1.20x1.40mm_HandSolder; LCSC Part (none) -> C95781; Part (none) -> RC0805FR-071KL; URL (none) -> https://www.lcsc.com/product-detail/Chip-Resistor-Surface-M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
- R5: value 10k -> 1M; footprint Resistor_SMD:R_0603_1608Metric -> Resistor_SMD:R_0805_2012Metric_Pad1.20x1.40mm_HandSolder; LCSC Part (none) -> C107700; Part (none) -> RC0805FR-071ML; URL (none) -> https://www.lcsc.com/product-detail/Chip-Resistor-Surface-M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
- R6: value 1k -> 5k1; footprint Resistor_SMD:R_0603_1608Metric -> Resistor_SMD:R_0805_2012Metric_Pad1.20x1.40mm_HandSolder; LCSC Part (none) -> C84375; Part (none) -> RC0805FR-075K1L; URL (none) -> https://www.lcsc.com/product-detail/Chip-Resistor-Surface-M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
Connections:
- net GND: now also R2.2, R5.2, R6.1, BT1.2 (-), C1.2, C10.2, C11.2, C12.2, C13.2, C14.2, C15.2, C16.2, C18.2, C19.2, C2.2, C20.2, C21.2, C3.2, C4.2, C5.2, C6.2, C8.2, C9.2, H1.1, H2.1, H3.1, H4.1, J1.3 (Pin_3), J2.A1 (GND), J2.A12 (GND), J2.B1 (GND), J2.B12 (GND), R7.1, U1.2 (GND), U2.10 (GND), U2.28 (GND), U3.4 (GND), U4.4 (GND), U6.2 (ADDR), U6.7 (R), U6.8 (VSS), U6.9 (VSS), U7.10 (GND@1), U7.12 (GND@2), U7.5 (GND@0), U7.7 (SA0), U8.2 (ADDR), U8.3 (GND), U8.7 (EXP), U9.4 (VSS)
- net LED: now reaches D2.1 (K)
- net LED: now also U2.22 (PA23/VDDIO/EXTINT[7]/X[11]/SERCOM3/PAD[1]/SERCOM5/PAD[1]/TC4/WO[1]/TCC0/WO[5]/USB/SOF1KHZ/GCLK_IO[7])
- net at D2.2 (A): now also R8.2
- net USB_VBUS_SENSE: now reaches R1.2
- net USB_VBUS_SENSE: now also R2.1, U2.25 (PA27/VDDIO/EXTINT[15]/GCLK_IO[0])
- net at R6.2: now also J2.A5 (CC1)
- net +3V0: now reaches R4.1
- net +3V0: now also R3.1, C10.1, C15.1, C16.1, C18.1, C19.1, C21.1, C3.1, C4.1, C8.1, C9.1, FB1.1, J1.2 (Pin_2), NT1.1, NT2.1, NT3.2, NT4.1, NT5.2, Q1.2 (S), R10.1, R8.1, R9.1, U1.1 (OUT), U2.30 (VDDIN), U3.8 (VCC)
- net ~RESET: now reaches R4.2
- net ~RESET: now also C6.1, J1.1 (Pin_1), U2.26 (~{RESET})
- net SWDCLK: now reaches R3.2
- net SWDCLK: now also J1.5 (Pin_5), U2.31 (PA30/VDDIO/EXTINT[10]/SERCOM1/PAD[2]/TCC1/WO[0]/SWCLK/GCLK_IO[0])
- net at R5.1: now also C12.1, D3.1 (GND), J2.S1 (SHIELD)
- net +3V3 renamed +5V
- net +5V: now also C5.1, D1.1 (K), D3.4 (VCC), Q1.1 (G), U1.3 (IN)
- new net: NT1.2, U4.8 (VCC)
- new net: F1.1, Q1.3 (D)
- new net: BT1.1 (+), F1.2
- new net: AE1.2, U9.2 (AC0)
- new net: AE1.1, U9.3 (AC1)
- new net: NT3.1, U9.8 (VCC)
- new net: C13.1, C14.1, FB1.2, U2.9 (VDDANA)
- new net: D1.2 (A), J2.A4 (VBUS), J2.A9 (VBUS), J2.B4 (VBUS), J2.B9 (VBUS)
- new net: NT5.1, U6.5 (VDD)
- new net: C11.1, U2.29 (VDDCORE)
- new net: NT2.2, U7.1 (VDDIO), U7.14 (VDD)
- new net: J2.B5 (CC2), R7.2
- new net: C20.1, U7.2 (BYP)
- new net: NT4.2, U8.1 (VDD)
- new net IMU_INT1: TP8.1, U2.8 (PA07/VDDANA/EXTINT[7]/AIN[7]/AIN[3]/Y[5]/SERCOM0/PAD[3]/TCC1/WO[1]/I2S/SD[0]), U7.9 (INT2)
- new net IMU_INT2: TP9.1, U2.7 (PA06/VDDANA/EXTINT[6]/AIN[6]/AIN[2]/Y[4]/SERCOM0/PAD[2]/TCC1/WO[0]), U7.11 (INT1)
- new net LIGHT_INT: TP11.1, U2.13 (PA10/VDDIO/EXTINT[10]/AIN[18]/X[2]/SERCOM0/PAD[2]/SERCOM2/PAD[2]/TCC1/WO[0]/TCC0/WO[2]/I2S/SCK[0]/GCLK_IO[4]), U8.5 (INT)
- new net MISO: U2.20 (PA19/VDDIO/EXTINT[3]/X[7]/SERCOM1/PAD[3]/SERCOM3/PAD[3]/TC3/WO[1]/TCC0/WO[3]/I2S/SD[0]/AC/CMP[1]), U3.2 (SO)
- new net MOSI: U2.17 (PA16/VDDIO/EXTINT[0]/X[4]/SERCOM1/PAD[0]/SERCOM3/PAD[0]/TCC2/WO[0]/TCC0/WO[6]/GCLK_IO[2]), U3.5 (SI)
- new net NFC_INT: TP6.1, U2.4 (PA03/VDDANA/EXTINT[3]/ADC/VREFADAC/VREFA/AIN[1]/Y[1]), U9.7 (GPO_(OD))
- new net SCK: U2.18 (PA17/VDDIO/EXTINT[1]/X[5]/SERCOM1/PAD[1]/SERCOM3/PAD[1]/TCC2/WO[1]/TCC0/WO[7]/GCLK_IO[3]), U3.6 (SCK)
- new net SCL: R10.2, TP2.1, U2.12 (PA09/VDDIO/EXTINT[9]/AIN[17]/X[1]/SERCOM0/PAD[1]/SERCOM2/PAD[1]/TCC0/WO[1]/TCC1/WO[3]/I2S/MCK[0]), U4.6 (SCL), U6.4 (SCL), U7.4 (SCL), U8.4 (SCL), U9.6 (SCL)
- new net SDA: R9.2, TP1.1, U2.11 (PA08/VDDIO/NMI/AIN[16]/X[0]/SERCOM0/PAD[0]/SERCOM2/PAD[0]/TCC0/WO[0]/TCC1/WO[2]/I2S/SD[1]), U4.5 (SDA), U6.1 (SDA), U7.6 (SDA), U8.6 (SDA), U9.5 (SDA)
- new net SWDIO: J1.8 (Pin_8), U2.32 (PA31/VDDIO/EXTINT[11]/SERCOM1/PAD[3]/TCC1/WO[1]/SWDIO)
- new net TEMP_INT: U2.6 (PA05/VDDANA/EXTINT[5]/AIN[5]/AIN[1]/Y[3]/SERCOM0/PAD[1]/TCC0/WO[1]), U6.3 (ALERT)
- new net USB_D+: D3.2 (I/O1), J2.A6 (D+), J2.B6 (D+), U2.24 (PA25/VDDIO/EXTINT[13]/SERCOM3/PAD[3]/SERCOM5/PAD[3]/TC5/WO[1]/TCC1/WO[3]/USB/DP)
- new net USB_D-: D3.3 (I/O2), J2.A7 (D-), J2.B7 (D-), U2.23 (PA24/VDDIO/EXTINT[12]/SERCOM3/PAD[2]/SERCOM5/PAD[2]/TC5/WO[0]/TCC1/WO[2]/USB/DM)
- new net XIN32: C1.1, U2.1 (PA00/VDDANA/EXTINT[0]/SERCOM1/PAD[0]/TCC2/WO[0]), Y1.1
- new net XOUT32: C2.1, U2.2 (PA01/VDDANA/EXTINT[1]/SERCOM1/PAD[1]/TCC2/WO[1]), Y1.2
- new net ~FLASH_CS: U2.19 (PA18/VDDIO/EXTINT[2]/X[6]/SERCOM1/PAD[2]/SERCOM3/PAD[2]/TC3/WO[0]/TCC0/WO[2]/AC/CMP[0]), U3.1 (~{CS})
- new net ~TEMP_RESET: U2.21 (PA22/VDDIO/EXTINT[6]/X[10]/SERCOM3/PAD[0]/SERCOM5/PAD[0]/TC4/WO[0]/TCC0/WO[4]/GCLK_IO[6]), U6.6 (~{RESET})
- no-connect marks 0 -> 14
Other:
- note added: "3-AXIS ACCELEROMETER"
- note added: "AMBIENT LIGHT SENSOR"
- note added: "Antenna design double-layer : AN5605"
- note added: "Antenna design: AN2972"
- note added: "D+/D- is differential pair Zdiff (differential impedance) is equal to 2 * Zodd, so a Zodd of 45 Ω gives us a Zdiff of 90 Ω"
- note added: "FTM Data exchange: AN4910"
- note added: "HARDWARE CRYPTO"
- note added: "NFC"
- note added: "NOR FLASH"
- note added: "PICKIT"
- note added: "POWER"
- note added: "ST25DV ultra-low power: AN5733"
- note added: "Should be 2V4+ flash, AT25DF is 2V6+"
- note added: "TEMPERATURE & HUMIDITY SENSOR"
- note added: "TODO: USB-C connector has mounting pins. The footprint should be updated accordingly."
- note added: "С=28.5pF equivalent L=4.9uH"
- note removed: "3.3V supply | GND | EN pin pulled HIGH via 10k | IO2 strapping to GND USB-C D+ D- to ESP32-C3 native USB pins I2C: SDA=GPIO8, SCL=GPIO9 | SPI: CLK=GPIO4, MOSI=GPIO6, MISO=GPIO2"
- note removed: "Cryo Sentinel — Intelligent Cold Chain Guardian"
- note removed: "Date: June 2026 | Rev: v2.0"
- note removed: "GPS MODULE (UART)"
- note removed: "I2C SENSORS (SDA=GPIO8, SCL=GPIO9)"
- note removed: "INDICATORS, BUZZER & TAMPER"
- note removed: "J1: JST-PH 2-pin LiPo connector (1000mAh 3.7V) J2: USB-C receptacle (TP4056 VBUS + ESP32 D+/D-) U8: TP4056 | USB-C VIN -> LiPo charge | 1A charge current | charge indicator LED U10: DW01A + FS8205 battery protection IC | overvoltage/overcurrent/reverse U11: AMS1117-3.3 | LiPo+ -> VBAT -> AMS1117 IN -> 3.3V -> all ICs D4: LED + R4(330ohm) battery indicator driven from GPIO15"
- note removed: "MCU: U1 — ESP32-C3-MINI-1"
- note removed: "POWER SYSTEM"
- note removed: "RGB LED (common cathode): GPIO12->R1(330)->D1(RED)->GND | GPIO13->R2(330)->D2(GRN)->GND | GPIO14->R3(330)->D3(BLU)->GND BUZZER: GPIO11->R6(1k)->Q1(2N2222 NPN BASE) | Q1_COLLECTOR->BZ1->3.3V | Q1_EMITTER->GND TAMPER: GPIO0->R5(10k)->3.3V (pullup) | PCB trace: GPIO0->lid_pad->GND via conductive trace Lid CLOSED: trace intact, GPIO0=LOW | Lid OPEN: trace broken, GPIO0=HIGH -> TAMPER EVENT"
- note removed: "SPI BUS (CLK=GPIO4, MOSI=GPIO6, MISO=GPIO2)"
- note removed: "U2: Sensirion SHT40 | Addr 0x44 | Temp/Humidity | VDD=3.3V | 100nF decoupling U3: Microchip ATECC608A | Addr 0x60 | HW Crypto ECC-P256 | 100nF decoupling U4: ST ST25DV04K | Addr 0x53 | NFC tag + I2C EEPROM | RF energy harvesting U9: Maxim MAX17048 | Addr 0x36 | LiPo Fuel Gauge | SDA/SCL shared bus"
- note removed: "U5: ADXL345 Accelerometer | CS=GPIO5 | ±16g range, full resolution, 100Hz ODR U6: SX1262 LoRa Module | CS=GPIO7, BUSY=GPIO3, DIO1=GPIO10, RST=GPIO1 865.0 MHz India band | SF9, BW125kHz | 14dBm TX | U.FL antenna connector NOTE: 50-ohm impedance-controlled trace required from module to U.FL J3: e-ink Display FPC 8-pin | CS=GPIO19, DC=GPIO18, RST=GPIO17, BUSY=GPIO16 1.54" 200x200 B/W | SSD1681 drive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"
- note removed: "U7: u-blox MAX-M10S | TX=GPIO21 (ESP RX), RX=GPIO20 (ESP TX) | 9600 baud Separate 3.3V LDO (U12 AMS1117-3.3) for GPS power domain LDO enable: GPIO controlled for switchable power-off Backup battery pad: CR1220 coin cell for RTC retention Passive antenna or active antenna with LNA bias"
- company: (none) -> apolisskyi
- title: (none) -> IoT risk logger
