File: hardware/cryosentinel.kicad_sch (KiCad schematic)
At the start: 63 parts, among them J1 Pickit 5 Conn, J2 USB Type-C, Q1 IRLML6401, U1 L78L33ABUTR, U2 ATSAMD21E18A-AU, U3 AT25DF321, U4 ATECC608A-MAHDA-S, U6 SHT30-DIS, U7 MMA8452QR1, U8 OPT3001DNPR, U9 ST25DV04K, Y1 SC-32S32.768

Commit message: hardware: complete CryoSentinel v2.0 schematic layout and 3D visualization
Parts:
- removed AE1: Antenna_Loop, footprints:ANT_NFC_30x40, symbol Device:Antenna_Loop
- removed BT1: 2xAAA, Battery:BatteryHolder_Keystone_2468_2xAAA, symbol Device:Battery
- removed C10, C13, C15, C16, C18, C19, C20, C21, C9: 100n, Capacitor_SMD:C_0805_2012Metric_Pad1.18x1.45mm_HandSolder, symbol Device:C
- removed C11, C14: 10u, Capacitor_SMD:C_0805_2012Metric_Pad1.18x1.45mm_HandSolder, symbol Device:C
- removed C12: 4n7, Capacitor_SMD:C_0805_2012Metric_Pad1.18x1.45mm_HandSolder, symbol Device:C
- removed D1: BAT60A, Diode_SMD:D_SOD-323_HandSoldering, symbol Diode:BAT60A
- removed D2: LED, LED_SMD:LED_0805_2012Metric_Pad1.15x1.40mm_HandSolder, symbol Device:LED
- removed D3: PRTR5V0U2X, Package_TO_SOT_SMD:SOT-143, symbol Power_Protection:PRTR5V0U2X
- removed F1: MSMF010 0.01A, Fuse:Fuse_1812_4532Metric_Pad1.30x3.40mm_HandSolder, symbol Device:Polyfuse
- removed FB1: 330, Resistor_SMD:R_0805_2012Metric_Pad1.20x1.40mm_HandSolder, symbol Device:FerriteBead_Small
- removed H1, H2, H3, H4: MountingHole_Pad, MountingHole:MountingHole_3.2mm_M3_Pad_Via, symbol Mechanical:MountingHole_Pad
- removed J1: Pickit 5 Conn, Connector_PinSocket_2.54mm:PinSocket_1x08_P2.54mm_Vertical, symbol Connector:Conn_01x08_Socket
- removed J2: USB Type-C, Connector_USB:USB_C_Receptacle_XKB_U262-16XN-4BVC11, symbol Connector:USB_C_Receptacle_USB2.0
- removed NT1, NT2, NT3, NT4, NT5: NetTie_2, NetTie:NetTie-2_SMD_Pad0.5mm, symbol Device:NetTie_2
- removed Q1: IRLML6401, Package_TO_SOT_SMD:SOT-23, symbol Device:Q_PMOS_GSD
- removed R10: 4k7, Resistor_SMD:R_0805_2012Metric_Pad1.20x1.40mm_HandSolder, symbol Device:R
- removed TP1, TP11, TP2, TP6, TP8, TP9: TestPoint_Probe, TestPoint:TestPoint_THTPad_D1.5mm_Drill0.7mm, symbol Connector:TestPoint_Probe
- removed U1: L78L33ABUTR, Package_TO_SOT_SMD:SOT-89-3_Handsoldering, symbol Regulator_Linear:L78L33_SOT89
- removed U2: ATSAMD21E18A-AU, Package_QFP:TQFP-32_7x7mm_P0.8mm, symbol ATSAMD21E17A-AUT:ATSAMD21E17A-AUT
- removed U3: AT25DF321, Package_SO:SOP-8_5.28x5.23mm_P1.27mm, symbol AT25DF041B-XMHN-B:AT25DF041B-XMHN-B
- removed U4: ATECC608A-MAHDA-S, Package_DFN_QFN:DFN-8-1EP_3x2mm_P0.5mm_EP1.3x1.5mm, symbol Security:ATECC608A-SSHDA
- removed U6: SHT30-DIS, Sensor_Humidity:Sensirion_DFN-8-1EP_2.5x2.5mm_P0.5mm_EP1.1x1.7mm, symbol Sensor_Humidity:SHT30-DIS
- removed U7: MMA8452QR1, Personal:XDCR_MMA8452QR1, symbol MMA8452Q:MMA8452Q
- removed U8: OPT3001DNPR, Personal:SON65P200X200X65-7N, symbol OPT3001DNPR:OPT3001DNPR
- removed U9: ST25DV04K, Package_SO:TSSOP-8_4.4x3mm_P0.65mm, symbol ST25DV64K-IER8T3:ST25DV64K-IER8T3
- removed Y1: SC-32S32.768, Crystal:Crystal_SMD_EuroQuartz_EQ161-2Pin_3.2x1.5mm_HandSoldering, symbol Device:Crystal
- added BZ1: Buzzer 3V Passive, symbol Device:Buzzer
- added C7: 4.7uF, symbol Device:C
- added J1: USB-C-16P, symbol Connector:USB_C_Receptacle_USB2.0_16P
- added J2: JST-PH-2, symbol Connector:Conn_01x02_Pin
- added J3: U.FL LoRa Antenna, symbol Connector:Conn_01x01_Pin
- added J4: U.FL GPS Antenna, symbol Connector:Conn_01x01_Pin
- added LED1: RGB LED CC, symbol Device:LED_ABGR
- added LED2: LED Battery, symbol Device:LED
- added PAD1: Tamper Pad A, symbol Connector:Conn_01x01_Pin
- added PAD2: Tamper Pad B, symbol Connector:Conn_01x01_Pin
- added Q1: MMBT2222, symbol Transistor_BJT:MMBT2222A
- added TP1: TP SDA, symbol Connector:Conn_01x01_Pin
- added TP2: TP SCL, symbol Connector:Conn_01x01_Pin
- added TP3: TP TX, symbol Connector:Conn_01x01_Pin
- added TP4: TP RX, symbol Connector:Conn_01x01_Pin
- added U1: ESP32-C3-MINI-1, symbol CryoSentinel_Custom:ESP32-C3-MINI-1
- added U10: 1.54in e-ink FPC-8, symbol Connector:Conn_01x08_Pin
- added U11: AT25DF321, symbol Memory_Flash:AT25SL321-U
- added U2: SHT40, symbol Sensor_Humidity:SHT31-DIS
- added U3: ATECC608A, symbol Security:ATECC608A-MAHDA
- added U4: ST25DV04K, symbol RF_NFC:ST25DV04K-IER8C3
- added U5: ADXL345, symbol Sensor_Motion:ADXL343
- added U6: SX1262, symbol RF_Module:RFM95W-868S2
- added U7: MAX-M10S, symbol RF_GPS:MAX-M10S
- added U8: MAX17048, symbol CryoSentinel_Custom:MAX17048
- added U9: TP4056, symbol CryoSentinel_Custom:TP4056
- C1, C2: value 22p -> 100nF; footprint Capacitor_SMD:C_0805_2012Metric_Pad1.18x1.45mm_HandSolder -> (none); LCSC Part C1804 -> (none); Part CL21C220JBANNNC -> (none); URL https://www.lcsc.com/product-detail/Multilayer-Ceramic-Capa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 -> (none)
- C3: value 22u -> 100nF; footprint Capacitor_SMD:C_1206_3216Metric_Pad1.33x1.80mm_HandSolder -> (none); LCSC Part C12891 -> (none); Part CL31A226KAHNNNE -> (none); URL https://www.lcsc.com/product-detail/Multilayer-Ceramic-Capa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 -> (none)
- C4: value 100n -> 100nF; footprint Capacitor_SMD:C_0805_2012Metric_Pad1.18x1.45mm_HandSolder -> (none); LCSC Part C1711 -> (none); Part CL21B104KBCNNNC -> (none); URL https://www.lcsc.com/product-detail/Multilayer-Ceramic-Capa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 -> (none)
- C5: value 10u -> 10uF; footprint Capacitor_SMD:C_0805_2012Metric_Pad1.18x1.45mm_HandSolder -> (none); LCSC Part C1713 -> (none); Part CL21A106KOQNNNE -> (none); URL https://www.lcsc.com/product-detail/Multilayer-Ceramic-Capa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 -> (none)
- C6, C8: value 100n -> 10uF; footprint Capacitor_SMD:C_0805_2012Metric_Pad1.18x1.45mm_HandSolder -> (none); LCSC Part C1711 -> (none); Part CL21B104KBCNNNC -> (none); URL https://www.lcsc.com/product-detail/Multilayer-Ceramic-Capa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 -> (none)
- R1, R2: value 10k -> 330R; footprint Resistor_SMD:R_0805_2012Metric_Pad1.20x1.40mm_HandSolder -> (none); LCSC Part C84376 -> (none); Part RC0805FR-0710KL -> (none); URL https://www.lcsc.com/product-detail/Chip-Resistor-Surface-M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 -> (none)
- R3: value 1k -> 330R; footprint Resistor_SMD:R_0805_2012Metric_Pad1.20x1.40mm_HandSolder -> (none); LCSC Part C95781 -> (none); Part RC0805FR-071KL -> (none); URL https://www.lcsc.com/product-detail/Chip-Resistor-Surface-M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 -> (none)
- R4: value 10k -> 4.7k; footprint Resistor_SMD:R_0805_2012Metric_Pad1.20x1.40mm_HandSolder -> (none); LCSC Part C84376 -> (none); Part RC0805FR-0710KL -> (none); URL https://www.lcsc.com/product-detail/Chip-Resistor-Surface-M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 -> (none)
- R5: value 1M -> 4.7k; footprint Resistor_SMD:R_0805_2012Metric_Pad1.20x1.40mm_HandSolder -> (none); LCSC Part C107700 -> (none); Part RC0805FR-071ML -> (none); URL https://www.lcsc.com/product-detail/Chip-Resistor-Surface-M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 -> (none)
- R6: value 5k1 -> 10k; footprint Resistor_SMD:R_0805_2012Metric_Pad1.20x1.40mm_HandSolder -> (none); LCSC Part C84375 -> (none); Part RC0805FR-075K1L -> (none); URL https://www.lcsc.com/product-detail/Chip-Resistor-Surface-M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 -> (none)
- R7: value 5k1 -> 1k; footprint Resistor_SMD:R_0805_2012Metric_Pad1.20x1.40mm_HandSolder -> (none); LCSC Part C84375 -> (none); Part RC0805FR-075K1L -> (none); URL https://www.lcsc.com/product-detail/Chip-Resistor-Surface-M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 -> (none)
- R8: value 1k -> 100k; footprint Resistor_SMD:R_0805_2012Metric_Pad1.20x1.40mm_HandSolder -> (none); LCSC Part C95781 -> (none); Part RC0805FR-071KL -> (none); URL https://www.lcsc.com/product-detail/Chip-Resistor-Surface-M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 -> (none)
- R9: value 4k7 -> 100k; footprint Resistor_SMD:R_0805_2012Metric_Pad1.20x1.40mm_HandSolder -> (none); LCSC Part C60816 -> (none); Part RC0805FR-074K7L -> (none); URL https://www.lcsc.com/product-detail/Chip-Resistor-Surface-M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 -> (none)
Connections:
- net +5V: no longer C5.1, R1.1
- net GND: no longer C1.2, C2.2, C3.2, C4.2, C5.2, C6.2, C8.2, R2.2, R5.2, R6.1, R7.1
- net MISO: now also U1.5 (IO2), U11.B2 (SO/IO1), U5.12 (SDO/ADDR), U6.2 (MISO)
- net MOSI: now also U1.9 (IO6), U10.6 (Pin_6), U11.D1 (SI/IO0), U5.13 (SDA/SDI/SDIO), U6.3 (MOSI)
- net SCL: now also U1.12 (IO9), U2.4 (SCL), U3.6 (SCL), U4.6 (SCL), U8.3 (SCL)
- net SDA: now also U1.11 (IO8), U2.1 (SDA), U3.5 (SDA), U4.5 (SDA), U8.5 (SDA); no longer R9.2
- removed net +3V0: C3.1, C4.1, C8.1, R3.1, R4.1, R8.1, R9.1
- net SWDCLK: no longer names the net of R3.2
- net USB_VBUS_SENSE: no longer names the net of R1.2
- net USB_VBUS_SENSE: no longer R2.1
- net XIN32: no longer names the net of C1.1
- net XOUT32: no longer names the net of C2.1
- net ~RESET: no longer names the net of R4.2
- net ~RESET: no longer C6.1
- new net: U7.1 (GND), U7.10 (GND), U7.12 (GND)
- new net: U2.8 (VSS), U2.9 (VSS)
- new net: J1.A1 (GND), J1.A12 (GND), J1.B1 (GND), J1.B12 (GND)
- new net: J1.A4 (VBUS), J1.A9 (VBUS), J1.B4 (VBUS), J1.B9 (VBUS)
- new net: U5.2 (GND), U5.4 (GND), U5.5 (GND)
- new net BUZZER: U1.15 (IO11)
- new net CLK: U1.7 (IO4), U10.5 (Pin_5), U11.C1 (SCK), U5.14 (SCL/SCLK), U6.4 (SCK)
- new net CS_ADXL: U1.8 (IO5), U5.7 (~{CS})
- new net CS_EINK: U1.23 (IO19), U10.4 (Pin_4)
- new net CS_FLASH: U1.19 (IO15), U11.A2 (~{CS})
- new net CS_LORA: U1.10 (IO7), U6.5 (NSS)
- new net EINK_BUSY: U1.20 (IO16), U10.1 (Pin_1)
- new net EINK_DC: U1.22 (IO18), U10.3 (Pin_3)
- new net EINK_RST: U1.21 (IO17), U10.2 (Pin_2)
- new net GPS_RX: U1.24 (IO20), U7.2 (TXD)
- new net GPS_TX: U1.25 (IO21), U7.3 (RXD)
- new net LED_B: U1.18 (IO14)
- new net LED_G: U1.17 (IO13)
- new net LED_R: U1.16 (IO12)
- new net LORA_BUSY: U1.6 (IO3), U6.14 (DIO0)
- new net LORA_DIO1: U1.13 (IO10), U6.15 (DIO1)
- new net LORA_RST: U1.4 (IO1), U6.6 (RESET)
- new net TAMPER: U1.3 (IO0)
- no-connect marks 14 -> 0
Other:
- note added: "BATTERY MANAGEMENT"
- note added: "E-INK DISPLAY"
- note added: "ESP32-C3 MCU"
- note added: "GPS MODULE"
- note added: "LORA MODULE"
- note added: "STATUS INDICATORS"
- note added: "TEMPERATURE & HUMIDITY"
- note removed: "AMBIENT LIGHT SENSOR"
- note removed: "Antenna design double-layer : AN5605"
- note removed: "Antenna design: AN2972"
- note removed: "D+/D- is differential pair Zdiff (differential impedance) is equal to 2 * Zodd, so a Zodd of 45 Ω gives us a Zdiff of 90 Ω"
- note removed: "FTM Data exchange: AN4910"
- note removed: "PICKIT"
- note removed: "ST25DV ultra-low power: AN5733"
- note removed: "Should be 2V4+ flash, AT25DF is 2V6+"
- note removed: "TEMPERATURE & HUMIDITY SENSOR"
- note removed: "TODO: USB-C connector has mounting pins. The footprint should be updated accordingly."
- note removed: "С=28.5pF equivalent L=4.9uH"
- company: apolisskyi -> (none)
- title: IoT risk logger -> (none)

Commit message: chore: Update schematic layout, dashboard screenshots, and README architecture diagrams
Connections:
- net +3V3: now also U1.1 (3V3), U1.2 (EN), U10.7 (Pin_7), U11.A1 (VCC), U11.B1 (~{HOLD}/IO3), U11.C2 (~{WP}/IO2), U2.5 (VDD), U2.8 (VSS), U2.9 (VSS), U8.5 (SDA)
- net +5V: now also U9.4 (VCC), U9.8 (CE)
- net BUZZER: now also U1.11 (IO8); no longer U1.15 (IO11)
- net CLK: now also U1.24 (IO20); no longer U1.7 (IO4), U5.14 (SCL/SCLK), U6.4 (SCK)
- net CS_ADXL: now also U1.6 (IO3); no longer U1.8 (IO5), U5.7 (~{CS})
- net CS_EINK: now also U1.19 (IO15); no longer U1.23 (IO19)
- net CS_FLASH: now also U1.25 (IO21); no longer U1.19 (IO15)
- net CS_LORA: now also U1.7 (IO4); no longer U1.10 (IO7), U6.5 (NSS)
- net EINK_BUSY: now also U1.16 (IO12); no longer U1.20 (IO16)
- net EINK_DC: now also U1.18 (IO14); no longer U1.22 (IO18)
- net EINK_RST: now also U1.17 (IO13); no longer U1.21 (IO17)
- net GND: now also J1.A1 (GND), J1.A12 (GND), J1.B1 (GND), J1.B12 (GND), J2.2 (Pin_2), U1.14 (GND), U10.8 (Pin_8), U11.D2 (GND), U2.2 (ADDR), U8.2 (GND), U9.1 (TEMP), U9.3 (GND)
- net GPS_RX: now also U1.20 (IO16); no longer U1.24 (IO20), U7.2 (TXD)
- net GPS_TX: now also U1.21 (IO17); no longer U1.25 (IO21), U7.3 (RXD)
- net LED_B: now also U1.15 (IO11); no longer U1.18 (IO14)
- net LED_G: now also U1.13 (IO10); no longer U1.17 (IO13)
- net LED_R: now also U1.12 (IO9); no longer U1.16 (IO12)
- net LORA_BUSY: now also U1.5 (IO2); no longer U1.6 (IO3), U6.14 (DIO0)
- net LORA_DIO1: now also U1.10 (IO7); no longer U1.13 (IO10), U6.15 (DIO1)
- net LORA_RST: no longer U6.6 (RESET)
- net MISO: now also U1.22 (IO18); no longer U1.5 (IO2), U5.12 (SDO/ADDR), U6.2 (MISO)
- net MOSI: now also U1.23 (IO19); no longer U1.9 (IO6), U5.13 (SDA/SDI/SDIO), U6.3 (MOSI)
- net SCL: now also U1.9 (IO6); no longer U1.12 (IO9), U3.6 (SCL), U4.6 (SCL)
- net SDA: now also U1.8 (IO5), U8.6 (~{ALRT}); no longer U1.11 (IO8), U3.5 (SDA), U4.5 (SDA), U8.5 (SDA)
- net VBAT: now also J2.1 (Pin_1), U8.1 (CELL), U9.5 (BAT)
- no-connect marks 0 -> 125
